Commit message: feat: (arm) add 'hardware_mode' parameter to select simulated or physical control
- hardware_mode:=mock_components for simulated, fake hardware (default)
- hardware_mode:=physical to talk to anchor and control the real arm

File: arm_moveit_config/config/ASTRA_Arm.ros2_control.xacro (robot description, xacro)
@@ -1,16 +1,22 @@
 <?xml version="1.0"?>
 <robot xmlns:xacro="http://www.ros.org/wiki/xacro">
-    <xacro:macro name="ASTRA_Arm_ros2_control" params="name initial_positions_file">
+    <xacro:macro name="ASTRA_Arm_ros2_control" params="name initial_positions_file hardware_mode">
         <xacro:property name="initial_positions" value="${xacro.load_yaml(initial_positions_file)['initial_positions']}"/>
         <ros2_control name="${name}" type="system">
             <hardware>
-                <!-- By default, set up controllers for simulation. This won't work on real hardware -->
-                <!-- <plugin>mock_components/GenericSystem</plugin> -->
-                <!-- <param name="calculate_dynamics">true</param> -->
-                <plugin>topic_based_ros2_control/TopicBasedSystem</plugin>
-                <param name="joint_commands_topic">/joint_commands</param>
-                <param name="joint_states_topic">/joint_states</param>
-                <param name="trigger_joint_command_threshold">1e-5</param>  <!-- Set to -1 to disable -->
-                <param name="sum_wrapped_joint_states">false</param>
+                <xacro:if value="${hardware_mode == 'mock_components'}">
+                    <!-- Use mock_components for a basic simulation. -->
+                    <plugin>mock_components/GenericSystem</plugin>
+                    <param name="calculate_dynamics">true</param>
+                    <param name="position_state_following_offset">0.0</param>
+                </xacro:if>
+                <xacro:unless value="${hardware_mode == 'mock_components'}">
+                    <!-- Use topic_based_ros2_control to interface with anchor and control real hardware -->
+                    <plugin>topic_based_ros2_control/TopicBasedSystem</plugin>
+                    <param name="joint_commands_topic">/joint_commands</param>
+                    <param name="joint_states_topic">/joint_states</param>
+                    <param name="trigger_joint_command_threshold">1e-5</param>  <!-- Set to -1 to disable -->
+                    <param name="sum_wrapped_joint_states">false</param>
+                </xacro:unless>
             </hardware>
             <joint name="Axis_0_Joint">

File: arm_moveit_config/config/ASTRA_Arm.urdf.xacro (robot description, xacro)
@@ -2,8 +2,9 @@
 <robot xmlns:xacro="http://www.ros.org/wiki/xacro" name="ASTRA_Arm">
     <xacro:arg name="initial_positions_file" default="initial_positions.yaml" />
+    <xacro:arg name="hardware_mode" default="mock_components" />
     <!-- Import ASTRA_Arm urdf file -->
     <xacro:include filename="$(find arm_description)/urdf/ASTRA_Arm.urdf" />
     <!-- Import control_xacro -->
     <xacro:include filename="ASTRA_Arm.ros2_control.xacro" />
-    <xacro:ASTRA_Arm_ros2_control name="FakeSystem" initial_positions_file="$(arg initial_positions_file)"/>
+    <xacro:ASTRA_Arm_ros2_control name="FakeSystem" initial_positions_file="$(arg initial_positions_file)" hardware_mode="$(arg hardware_mode)"/>
 </robot>
