Commit message: refactor!: unify hardware_mode behavior

File: arm_moveit_config/config/ASTRA_Arm.ros2_control.xacro (robot description, xacro)
@@ -3,81 +3,82 @@
     <xacro:macro name="ASTRA_Arm_ros2_control" params="name initial_positions_file hardware_mode">
         <xacro:property name="initial_positions" value="${xacro.load_yaml(initial_positions_file)['initial_positions']}"/>
-        <ros2_control name="${name}" type="system">
-            <hardware>
-                <xacro:if value="${hardware_mode == 'mock_components'}">
-                    <!-- Use mock_components for a basic simulation. -->
-                    <plugin>mock_components/GenericSystem</plugin>
-                    <param name="calculate_dynamics">true</param>
-                    <param name="position_state_following_offset">0.0</param>
-                </xacro:if>
-                <xacro:if value="${hardware_mode == 'gazebo'}">
-                    <plugin>gz_ros2_control/GazeboSimSystem</plugin>
-                </xacro:if>
-                <xacro:if value="${hardware_mode == 'physical'}">
-                    <!-- Use topic_based_ros2_control to interface with anchor and control real hardware -->
-                    <plugin>topic_based_ros2_control/TopicBasedSystem</plugin>
-                    <param name="joint_commands_topic">/arm/joint_commands</param>
-                    <param name="joint_states_topic">/joint_states</param>
-                    <param name="trigger_joint_command_threshold">1e-5</param>  <!-- Set to -1 to disable -->
-                    <param name="sum_wrapped_joint_states">false</param>
-                </xacro:if>
-            </hardware>
-            <joint name="axis_0_joint">
-                <!-- <command_interface name="position"/> -->
-                <command_interface name="velocity"/>
-                <state_interface name="position">
-                  <param name="initial_value">${initial_positions['axis_0_joint']}</param>
-                </state_interface>
-                <state_interface name="velocity"/>
-            </joint>
-            <joint name="axis_1_joint">
-                <!-- <command_interface name="position"/> -->
-                <command_interface name="velocity"/>
-                <state_interface name="position">
-                  <param name="initial_value">${initial_positions['axis_1_joint']}</param>
-                </state_interface>
-                <state_interface name="velocity"/>
-            </joint>
-            <joint name="axis_2_joint">
-                <!-- <command_interface name="position"/> -->
-                <command_interface name="velocity"/>
-                <state_interface name="position">
-                  <param name="initial_value">${initial_positions['axis_2_joint']}</param>
-                </state_interface>
-                <state_interface name="velocity"/>
-            </joint>
-            <joint name="axis_3_joint">
-                <!-- <command_interface name="position"/> -->
-                <command_interface name="velocity"/>
-                <state_interface name="position">
-                  <param name="initial_value">${initial_positions['axis_3_joint']}</param>
-                </state_interface>
-                <state_interface name="velocity"/>
-            </joint>
-            <joint name="wrist_yaw_joint">
-                <!-- <command_interface name="position"/> -->
-                <command_interface name="velocity"/>
-                <state_interface name="position">
-                  <param name="initial_value">${initial_positions['wrist_yaw_joint']}</param>
-                </state_interface>
-                <state_interface name="velocity"/>
-            </joint>
-            <joint name="wrist_roll_joint">
-                <!-- <command_interface name="position"/> -->
-                <command_interface name="velocity"/>
-                <state_interface name="position">
-                  <param name="initial_value">${initial_positions['wrist_roll_joint']}</param>
-                </state_interface>
-                <state_interface name="velocity"/>
-            </joint>
-            <joint name="ef_gripper_left_joint">
-                <!-- <command_interface name="position"/> -->
-                <command_interface name="velocity"/>
-                <state_interface name="position">
-                  <param name="initial_value">${initial_positions['ef_gripper_left_joint']}</param>
-                </state_interface>
-                <state_interface name="velocity"/>
-            </joint>
-        </ros2_control>
+        <!-- Reject an unrecognized hardware_mode. list.index() raises ValueError on a bad value. -->
+        <xacro:if value="${['preview', 'gazebo', 'physical'].index(hardware_mode) >= 0}">
+            <!-- unreachable body: valid modes evaluate True; an invalid one raises above -->
+        </xacro:if>
+        <!-- preview = geometry only; omit ros2_control (RSP/RViz ignore these tags anyway). -->
+        <xacro:unless value="${hardware_mode == 'preview'}">
+            <ros2_control name="${name}" type="system">
+                <hardware>
+                    <xacro:if value="${hardware_mode == 'gazebo'}">
+                        <plugin>gz_ros2_control/GazeboSimSystem</plugin>
+                    </xacro:if>
+                    <xacro:if value="${hardware_mode == 'physical'}">
+                        <!-- Use topic_based_ros2_control to interface with anchor and control real hardware -->
+                        <plugin>topic_based_ros2_control/TopicBasedSystem</plugin>
+                        <param name="joint_commands_topic">/arm/joint_commands</param>
+                        <param name="joint_states_topic">/joint_states</param>
+                        <param name="trigger_joint_command_threshold">1e-5</param>  <!-- Set to -1 to disable -->
+                        <param name="sum_wrapped_joint_states">false</param>
+                    </xacro:if>
+                </hardware>
+                <joint name="axis_0_joint">
+                    <!-- <command_interface name="position"/> -->
+                    <command_interface name="velocity"/>
+                    <state_interface name="position">
+                      <param name="initial_value">${initial_positions['axis_0_joint']}</param>
+                    </state_interface>
+                    <state_interface name="velocity"/>
+                </joint>
+                <joint name="axis_1_joint">
+                    <!-- <command_interface name="position"/> -->
+                    <command_interface name="velocity"/>
+                    <state_interface name="position">
+                      <param name="initial_value">${initial_positions['axis_1_joint']}</param>
+                    </state_interface>
+                    <state_interface name="velocity"/>
+                </joint>
+                <joint name="axis_2_joint">
+                    <!-- <command_interface name="position"/> -->
+                    <command_interface name="velocity"/>
+                    <state_interface name="position">
+                      <param name="initial_value">${initial_positions['axis_2_joint']}</param>
+                    </state_interface>
+                    <state_interface name="velocity"/>
+                </joint>
+                <joint name="axis_3_joint">
+                    <!-- <command_interface name="position"/> -->
+                    <command_interface name="velocity"/>
+                    <state_interface name="position">
+                      <param name="initial_value">${initial_positions['axis_3_joint']}</param>
+                    </state_interface>
+                    <state_interface name="velocity"/>
+                </joint>
+                <joint name="wrist_yaw_joint">
+                    <!-- <command_interface name="position"/> -->
+                    <command_interface name="velocity"/>
+                    <state_interface name="position">
+                      <param name="initial_value">${initial_positions['wrist_yaw_joint']}</param>
+                    </state_interface>
+                    <state_interface name="velocity"/>
+                </joint>
+                <joint name="wrist_roll_joint">
+                    <!-- <command_interface name="position"/> -->
+                    <command_interface name="velocity"/>
+                    <state_interface name="position">
+                      <param name="initial_value">${initial_positions['wrist_roll_joint']}</param>
+                    </state_interface>
+                    <state_interface name="velocity"/>
+                </joint>
+                <joint name="ef_gripper_left_joint">
+                    <!-- <command_interface name="position"/> -->
+                    <command_interface name="velocity"/>
+                    <state_interface name="position">
+                      <param name="initial_value">${initial_positions['ef_gripper_left_joint']}</param>
+                    </state_interface>
+                    <state_interface name="velocity"/>
+                </joint>
+            </ros2_control>
+        </xacro:unless>
         <!-- Gazebo ros2_control Plugin tag omitted, arm cannot be ran w/o Core in Gazebo -->
     </xacro:macro>

File: core_description/urdf/core_description.xacro (robot description, xacro)
@@ -1,8 +1,11 @@
 <?xml version="1.0"?>
 <robot xmlns:xacro="http://www.ros.org/wiki/xacro" name="core_rover">
-  <xacro:arg name="hardware_mode" default="gazebo"/>
-  <xacro:arg name="omit_gz_ros2_control" default="false"/>
+  <xacro:arg name="hardware_mode" default="preview"/>
+  <!-- Tells Core to add its own gz_ros2_control plugin. Default false so combining into
+       rover_description doesn't add a second one (double controller_manager);
+       standalone core sim sets it true. -->
+  <xacro:arg name="add_core_gz_ros2_control" default="false"/>
   <xacro:include filename="core_description.urdf"/>
   <xacro:include filename="ros2_control.xacro"/>
-  <xacro:core_ros2_control hardware_mode="$(arg hardware_mode)" omit_gz_ros2_control="$(arg omit_gz_ros2_control)"/>
+  <xacro:core_ros2_control hardware_mode="$(arg hardware_mode)" add_core_gz_ros2_control="$(arg add_core_gz_ros2_control)"/>
 </robot>

File: core_description/urdf/ros2_control.xacro (robot description, xacro)
@@ -1,44 +1,51 @@
 <?xml version="1.0"?>
 <robot xmlns:xacro="http://www.ros.org/wiki/xacro">
-    <xacro:macro name="core_ros2_control" params="hardware_mode omit_gz_ros2_control">
-        <ros2_control name="CoreSystem" type="system">
-            <hardware>
-                <xacro:if value="${hardware_mode == 'gazebo'}">
-                    <plugin>gz_ros2_control/GazeboSimSystem</plugin>
-                </xacro:if>
-                <xacro:unless value="${hardware_mode == 'gazebo'}">
-                    <!-- Use topic_based_ros2_control to interface with anchor and control real hardware -->
-                    <plugin>topic_based_ros2_control/TopicBasedSystem</plugin>
-                    <param name="joint_commands_topic">/core/joint_commands</param>
-                    <param name="joint_states_topic">/joint_states</param>
-                    <param name="trigger_joint_command_threshold">-1</param>  <!-- Set to -1 to disable -->
-                    <param name="sum_wrapped_joint_states">true</param>
-                </xacro:unless>
-            </hardware>
-            <joint name="left_suspension_joint">
-                <state_interface name="position"/>
-            </joint>
-            <joint name="bl_wheel_joint">
-                <command_interface name="velocity"/>
-                <state_interface name="velocity"/>
-                <state_interface name="position"/>
-            </joint>
-            <joint name="br_wheel_joint">
-                <command_interface name="velocity"/>
-                <state_interface name="velocity"/>
-                <state_interface name="position"/>
-            </joint>
-            <joint name="fl_wheel_joint">
-                <command_interface name="velocity"/>
-                <state_interface name="velocity"/>
-                <state_interface name="position"/>
-            </joint>
-            <joint name="fr_wheel_joint">
-                <command_interface name="velocity"/>
-                <state_interface name="velocity"/>
-                <state_interface name="position"/>
-            </joint>
-        </ros2_control>
-        <xacro:unless value="${omit_gz_ros2_control}">
+    <xacro:macro name="core_ros2_control" params="hardware_mode add_core_gz_ros2_control">
+        <!-- Reject an unrecognized hardware_mode. list.index() raises ValueError on a bad value. -->
+        <xacro:if value="${['preview', 'gazebo', 'physical'].index(hardware_mode) >= 0}">
+            <!-- unreachable body: valid modes evaluate True; an invalid one raises above -->
+        </xacro:if>
+        <!-- preview = geometry only; omit ros2_control (RSP/RViz ignore these tags anyway). -->
+        <xacro:unless value="${hardware_mode == 'preview'}">
+            <ros2_control name="CoreSystem" type="system">
+                <hardware>
+                    <xacro:if value="${hardware_mode == 'gazebo'}">
+                        <plugin>gz_ros2_control/GazeboSimSystem</plugin>
+                    </xacro:if>
+                    <xacro:if value="${hardware_mode == 'physical'}">
+                        <!-- Use topic_based_ros2_control to interface with anchor and control real hardware -->
+                        <plugin>topic_based_ros2_control/TopicBasedSystem</plugin>
+                        <param name="joint_commands_topic">/core/joint_commands</param>
+                        <param name="joint_states_topic">/joint_states</param>
+                        <param name="trigger_joint_command_threshold">-1</param>  <!-- Set to -1 to disable -->
+                        <param name="sum_wrapped_joint_states">true</param>
+                    </xacro:if>
+                </hardware>
+                <joint name="left_suspension_joint">
+                    <state_interface name="position"/>
+                </joint>
+                <joint name="bl_wheel_joint">
+                    <command_interface name="velocity"/>
+                    <state_interface name="velocity"/>
+                    <state_interface name="position"/>
+                </joint>
+                <joint name="br_wheel_joint">
+                    <command_interface name="velocity"/>
+                    <state_interface name="velocity"/>
+                    <state_interface name="position"/>
+                </joint>
+                <joint name="fl_wheel_joint">
+                    <command_interface name="velocity"/>
+                    <state_interface name="velocity"/>
+                    <state_interface name="position"/>
+                </joint>
+                <joint name="fr_wheel_joint">
+                    <command_interface name="velocity"/>
+                    <state_interface name="velocity"/>
+                    <state_interface name="position"/>
+                </joint>
+            </ros2_control>
+        </xacro:unless>
+        <xacro:if value="${add_core_gz_ros2_control}">
             <xacro:if value="${hardware_mode == 'gazebo'}">
                 <gazebo>
@@ -52,5 +59,5 @@
                 </gazebo>
             </xacro:if>
-        </xacro:unless>
+        </xacro:if>
     </xacro:macro>
 </robot>

File: rover_description/urdf/rover_description.xacro (robot description, xacro)
@@ -1,5 +1,17 @@
 <?xml version="1.0"?>
+<!-- Renaming this robot can quietly break MoveIt2: the name is coupled to several MoveIt2
+     config filenames across several files in strange, undocumented ways. If you rename,
+     change it in all of these together:
+       - this <robot name> attribute
+       - the <robot name> in arm_moveit_config/config/ASTRA_Arm.srdf and ASTRA_Arm.urdf.xacro
+       - the MoveItConfigsBuilder(...) arg and the ASTRA_Arm.* filenames it resolves, in
+         arm_moveit_config/launch/moveit2.launch.py
+       - the paths recorded in arm_moveit_config/.setup_assistant
+     The inter-dependency theoretically comes from MoveIt2's SRDF loader and its config builder. -->
 <robot xmlns:xacro="http://www.ros.org/wiki/xacro" name="ASTRA_Arm">
-    <xacro:arg name="hardware_mode" default="mock_components" />
+    <xacro:arg name="hardware_mode" default="preview" />
+    <!-- rover_description owns the combined gz_ros2_control plugin below, so suppress
+         core's by default; standalone core sim sets it true. -->
+    <xacro:arg name="add_core_gz_ros2_control" default="false" />
     <!-- Import Arm Xacro file -->
     <xacro:include filename="$(find arm_moveit_config)/config/ASTRA_Arm.urdf.xacro" />
@@ -16,14 +28,18 @@
             link="arm_base_link" />
     </joint>
-    <gazebo>
-        <plugin filename="gz_ros2_control-system" name="gz_ros2_control::GazeboSimROS2ControlPlugin">
-            <parameters>$(find core_description)/config/ros2_controllers.yaml</parameters>
-            <parameters>$(find arm_moveit_config)/config/ros2_controllers.yaml</parameters>
-            <ros>
-                <remapping>/diff_controller/cmd_vel_unstamped:=/core/control/cmd_vel</remapping>
-                <remapping>/diff_controller/odom:=/core/feedback/wheel_odom</remapping>
-                <remapping>/hand_controller/commands:=/arm/control/ik_gripper</remapping>
-            </ros>
-        </plugin>
-    </gazebo>
+    <!-- Declare a singular ros2_control plugin for Gazebo with the controllers required
+         for both Core and Arm. -->
+    <xacro:if value="${'$(arg hardware_mode)' == 'gazebo'}">
+        <gazebo>
+            <plugin filename="gz_ros2_control-system" name="gz_ros2_control::GazeboSimROS2ControlPlugin">
+                <parameters>$(find core_description)/config/ros2_controllers.yaml</parameters>
+                <parameters>$(find arm_moveit_config)/config/ros2_controllers.yaml</parameters>
+                <ros>
+                    <remapping>/diff_controller/cmd_vel_unstamped:=/core/control/cmd_vel</remapping>
+                    <remapping>/diff_controller/odom:=/core/feedback/wheel_odom</remapping>
+                    <remapping>/hand_controller/commands:=/arm/control/ik_gripper</remapping>
+                </ros>
+            </plugin>
+        </gazebo>
+    </xacro:if>
 </robot>
