Commit message: feat: (core) rewrite, add topic_based to control xacro
Rewrote everything, should still work :)
Added hardware_mode parameter to launch files. 'preview', 'gazebo', and 'physical' control behavior of display.launch.py and robot_state_publisher.launch.py

File: core_description/urdf/core_description.xacro (robot description, xacro)
@@ -1,5 +1,7 @@
 <?xml version="1.0"?>
 <robot xmlns:xacro="http://www.ros.org/wiki/xacro" name="core_rover">
+  <xacro:arg name="hardware_mode" default="gazebo"/>
   <xacro:include filename="core_rover.urdf"/>
   <xacro:include filename="ros2_control.xacro"/>
+  <xacro:core_ros2_control hardware_mode="$(arg hardware_mode)"/>
 </robot>

File: core_description/urdf/ros2_control.xacro (robot description, xacro)
@@ -1,39 +1,53 @@
 <?xml version="1.0"?>
 <robot xmlns:xacro="http://www.ros.org/wiki/xacro">
-    <ros2_control name="GazeboSystem" type="system">
-        <hardware>
-            <plugin>gz_ros2_control/GazeboSimSystem</plugin>
-        </hardware>
-        <joint name="left_suspension_joint">
-            <state_interface name="position"/>
-        </joint>
-        <joint name="bl_wheel_joint">
-            <command_interface name="velocity"/>
-            <state_interface name="velocity"/>
-            <state_interface name="position"/>
-        </joint>
-        <joint name="br_wheel_joint">
-            <command_interface name="velocity"/>
-            <state_interface name="velocity"/>
-            <state_interface name="position"/>
-        </joint>
-        <joint name="fl_wheel_joint">
-            <command_interface name="velocity"/>
-            <state_interface name="velocity"/>
-            <state_interface name="position"/>
-        </joint>
-        <joint name="fr_wheel_joint">
-            <command_interface name="velocity"/>
-            <state_interface name="velocity"/>
-            <state_interface name="position"/>
-        </joint>
-    </ros2_control>
-    <gazebo>
-        <plugin filename="gz_ros2_control-system" name="gz_ros2_control::GazeboSimROS2ControlPlugin">
-            <parameters>$(find core_description)/config/ros2_controllers.yaml</parameters>
-            <ros>
-                <remapping>/diff_controller/cmd_vel_unstamped:=/core/twist</remapping>
-            </ros>
-        </plugin>
-    </gazebo>
+    <xacro:macro name="core_ros2_control" params="hardware_mode">
+        <ros2_control name="CoreSystem" type="system">
+            <hardware>
+                <xacro:if value="${hardware_mode == 'gazebo'}">
+                    <plugin>gz_ros2_control/GazeboSimSystem</plugin>
+                </xacro:if>
+                <xacro:unless value="${hardware_mode == 'gazebo'}">
+                    <!-- Use topic_based_ros2_control to interface with anchor and control real hardware -->
+                    <plugin>topic_based_ros2_control/TopicBasedSystem</plugin>
+                    <param name="joint_commands_topic">/joint_commands</param>
+                    <param name="joint_states_topic">/joint_states</param>
+                    <param name="trigger_joint_command_threshold">1e-5</param>  <!-- Set to -1 to disable -->
+                    <param name="sum_wrapped_joint_states">true</param>
+                </xacro:unless>
+            </hardware>
+            <joint name="left_suspension_joint">
+                <state_interface name="position"/>
+            </joint>
+            <joint name="bl_wheel_joint">
+                <command_interface name="velocity"/>
+                <state_interface name="velocity"/>
+                <state_interface name="position"/>
+            </joint>
+            <joint name="br_wheel_joint">
+                <command_interface name="velocity"/>
+                <state_interface name="velocity"/>
+                <state_interface name="position"/>
+            </joint>
+            <joint name="fl_wheel_joint">
+                <command_interface name="velocity"/>
+                <state_interface name="velocity"/>
+                <state_interface name="position"/>
+            </joint>
+            <joint name="fr_wheel_joint">
+                <command_interface name="velocity"/>
+                <state_interface name="velocity"/>
+                <state_interface name="position"/>
+            </joint>
+        </ros2_control>
+        <xacro:if value="${hardware_mode == 'gazebo'}">
+            <gazebo>
+                <plugin filename="gz_ros2_control-system" name="gz_ros2_control::GazeboSimROS2ControlPlugin">
+                    <parameters>$(find core_description)/config/ros2_controllers.yaml</parameters>
+                    <ros>
+                        <remapping>/diff_controller/cmd_vel_unstamped:=/core/twist</remapping>
+                    </ros>
+                </plugin>
+            </gazebo>
+        </xacro:if>
+    </xacro:macro>
 </robot>
