Commit message: refactor(core): re-export Core URDF
Reduces the size of core_description from 35M to 13M, and updates it to the current main assembly. Adds models from CAD for the antenna mast, camera mount, GPS antenna, and ZED. Also cleans up the base_link/dummy_base_link situation; base_link is now in the correct coordinate frame directly from CAD. Retains Gazebo sensor functionality.

File: core_description/urdf/core_description.urdf (robot description, URDF)
Before this commit: robot core_description, 12 links, 11 joints
Links:
- removed link averaging_bar
- removed link bl_wheel
- removed link br_wheel
- removed link dummy_base_link
- removed link fl_wheel
- removed link fr_wheel
- removed link left_suspension_member
- removed link right_suspension_member
- added link averaging_bar_link, mass 0.83085; collision mesh filename=package://core_description/meshes/averaging_bar_link.STL; visual mesh filename=package://core_description/meshes/averaging_bar_link.STL
- added link bl_wheel_link, mass 5.1003; collision mesh filename=package://core_description/meshes/bl_wheel_link.STL; visual mesh filename=package://core_description/meshes/bl_wheel_link.STL
- added link br_wheel_link, mass 5.1003; collision mesh filename=package://core_description/meshes/br_wheel_link.STL; visual mesh filename=package://core_description/meshes/br_wheel_link.STL
- added link fl_wheel_link, mass 5.1003; collision mesh filename=package://core_description/meshes/fl_wheel_link.STL; visual mesh filename=package://core_description/meshes/fl_wheel_link.STL
- added link fr_wheel_link, mass 5.1003; collision mesh filename=package://core_description/meshes/fr_wheel_link.STL; visual mesh filename=package://core_description/meshes/fr_wheel_link.STL
- added link left_suspension_link, mass 2.3189; collision mesh filename=package://core_description/meshes/left_suspension_link.STL; visual mesh filename=package://core_description/meshes/left_suspension_link.STL
- added link right_suspension_link, mass 2.3189; collision mesh filename=package://core_description/meshes/right_suspension_link.STL; visual mesh filename=package://core_description/meshes/right_suspension_link.STL
- added link zed_camera_link, mass 0.17032; collision mesh filename=package://core_description/meshes/zed_camera_link.STL; visual mesh filename=package://core_description/meshes/zed_camera_link.STL
- link base_link: mass 75.3855391061812 -> 72.183
- link core_gps_antenna_link: mass 0.05 -> 0; geometry collision mesh filename=package://core_description/meshes/core_gps_antenna_link.STL; visual mesh filename=package://core_description/meshes/core_gps_antenna_link.STL
Joints:
- removed joint dummy_base_link_joint
- added joint zed_camera_joint: type fixed, parent base_link, child zed_camera_link, origin xyz=0.30801 -0.00055649 0.041848 rpy=0 0 1.5708, axis 0 0 0
- joint averaging_bar_joint: child averaging_bar -> averaging_bar_link; limit lower=-0.38 upper=0.38 effort=50 velocity=1.5 -> lower=-0.38 upper=0.38 effort=0 velocity=0; origin xyz=0 -0.23362 -0.0508 rpy=0 -0.0060774 -3.1416 -> xyz=0.3066 -0.009525 0.075057 rpy=3.1416 0.003802 -1.5708
- joint bl_wheel_joint: child bl_wheel -> bl_wheel_link; origin xyz=0.41838 -0.17155 0.12984 rpy=1.5769 -1.5708 0 -> xyz=0.39101 -0.14546 0.1297 rpy=2.2133 -1.5708 -1.5622; parent left_suspension_member -> left_suspension_link
- joint br_wheel_joint: child br_wheel -> br_wheel_link; origin xyz=-0.41838 -0.17155 0.12984 rpy=0.52965 -1.5708 0 -> xyz=0.40478 0.14243 -0.21002 rpy=0.89286 1.5708 0; parent right_suspension_member -> right_suspension_link
- joint core_camera_joint: origin xyz=0 -0.265 -0.035 rpy=0 0 -1.5707963267948966 -> xyz=0.348 -0.038 0.085 rpy=0 0.262 0
- joint core_embedded_imu_joint: origin xyz=0 -0.26 0 rpy=0 0 -1.5707963267948966 -> xyz=0.1 -0.23 0.135 rpy=0 0 0
- joint core_gps_antenna_joint: axis (none) -> 0 0 0; origin xyz=0.25 0.475 0.6 rpy=0 0 -1.5707963267948966 -> xyz=-0.42556 0.1677 1.4846 rpy=0 0 -1.5708
- joint fl_wheel_joint: child fl_wheel -> fl_wheel_link; origin xyz=-0.418377874454344 -0.171553199039643 0.129841324042317 rpy=0.529654981264331 -1.5707963267949 0 -> xyz=-0.39101 -0.14546 0.1297 rpy=-3.0652 -1.5708 -1.5622; parent left_suspension_member -> left_suspension_link
- joint fr_wheel_joint: axis -1 0 0 -> 0 -1 0; child fr_wheel -> fr_wheel_link; origin xyz=0.41838 -0.17155 0.12984 rpy=1.5769 -1.5708 0 -> xyz=-0.16048 -0.39797 -0.12125 rpy=-1.5708 0 -1.459; parent right_suspension_member -> right_suspension_link
- joint left_suspension_joint: axis 0 0 -1 -> 0 0 1; child left_suspension_member -> left_suspension_link; limit lower=-0.38 upper=0.38 effort=50 velocity=1.5 -> lower=-0.38 upper=0.38 effort=0 velocity=0; origin xyz=0.33067 0.028531 -0.15443 rpy=1.5708 0 1.5708 -> xyz=0.025669 0.29798 -0.059879 rpy=1.5708 0.0086 3.1416
- joint right_suspension_joint: child right_suspension_member -> right_suspension_link; limit lower=-0.38 upper=0.38 effort=50 velocity=1.5 -> lower=-0.38 upper=0.38 effort=0 velocity=0; origin xyz=-0.33067 0.028531 -0.15443 rpy=1.5708 0 -1.5708 -> xyz=0.0254 -0.23671 -0.028575 rpy=1.5708 0.76291 3.1416

File: core_description/urdf/core_description.xacro (robot description, xacro)
@@ -3,5 +3,5 @@
   <xacro:arg name="hardware_mode" default="gazebo"/>
   <xacro:arg name="omit_gz_ros2_control" default="false"/>
-  <xacro:include filename="core_rover.urdf"/>
+  <xacro:include filename="core_description.urdf"/>
   <xacro:include filename="ros2_control.xacro"/>
   <xacro:core_ros2_control hardware_mode="$(arg hardware_mode)" omit_gz_ros2_control="$(arg omit_gz_ros2_control)"/>

File: rover_description/urdf/rover_description.xacro (robot description, xacro)
@@ -9,6 +9,6 @@
     <joint name="arm_core_joint" type="fixed">
         <origin
-            xyz="-0.03 -0.075 0.1"
-            rpy="0 0 0" />
+            xyz="0.13 -0.035 0.227"
+            rpy="0 0 1.5708" />
         <parent
             link="base_link" />
