Commit message: feat: add IMU and GPS antenna to URDF

File: core_description/urdf/core_rover.urdf (robot description, URDF)
Before this commit: robot core_description, 9 links, 8 joints
Links:
- added link core_embedded_imu_link, mass 0.003; visual box size=0.02 0.027 0.004
- added link core_gps_antenna_link, mass 0.05; visual box size=0.05 0.05 0.02
Joints:
- added joint core_embedded_imu_joint: type fixed, parent base_link, child core_embedded_imu_link, origin xyz=0 -0.26 0 rpy=0 0 -1.5707963267948966
- added joint core_gps_antenna_joint: type fixed, parent base_link, child core_gps_antenna_link, origin xyz=0.25 0.475 0.6 rpy=0 0 -1.5707963267948966

Commit message: fix(core): Gazebo no longer hangs on launch

File: core_description/urdf/core_rover.urdf (robot description, URDF)
Before this commit: robot core_description, 11 links, 10 joints
Links:
- link dummy_base_link: mass None -> 0.001
Joints:
- joint averaging_bar_joint: limit lower=-0.38 upper=0.38 effort=0 velocity=0 -> lower=-0.38 upper=0.38 effort=50 velocity=1.5
- joint left_suspension_joint: limit lower=-0.38 upper=0.38 effort=0 velocity=0 -> lower=-0.38 upper=0.38 effort=50 velocity=1.5
- joint right_suspension_joint: limit lower=-0.38 upper=0.38 effort=0 velocity=0 -> lower=-0.38 upper=0.38 effort=50 velocity=1.5

Commit message: feat(core): add camera to Gazebo

File: core_description/urdf/core_rover.urdf (robot description, URDF)
Before this commit: robot core_description, 11 links, 10 joints
Links:
- added link core_camera_link, mass 0.13; visual box size=0.02 0.034 0.034
Joints:
- added joint core_camera_joint: type fixed, parent base_link, child core_camera_link, origin xyz=0 -0.265 -0.035 rpy=0 0 -1.5707963267948966

Commit message: remove suspension joint limits

File: core_description/urdf/core_rover.urdf (robot description, URDF)
Before this commit: robot core_description, 12 links, 11 joints
Joints:
- joint left_suspension_joint: limit lower=-0.38 upper=0.38 effort=50 velocity=1.5 -> lower=0 upper=0 effort=50 velocity=1.5
- joint right_suspension_joint: limit lower=-0.38 upper=0.38 effort=50 velocity=1.5 -> lower=0 upper=0 effort=50 velocity=1.5
