Commit message: refactor!: formalize Arm URDF joint and link names

File: arm_description/urdf/ASTRA_Arm.urdf (robot description, URDF)
Before this commit: robot ASTRA_Arm, 9 links, 8 joints
Links:
- removed link Axis_0_Plate
- removed link Axis_1_Segment
- removed link Axis_2_Segment
- removed link Diff_Carrier
- removed link EF_Gripper_Left
- removed link EF_Gripper_Right
- removed link End_Effector
- removed link Wrist
- added link axis_0_link, mass 2.045; collision mesh filename=package://arm_description/meshes/axis_0_link.STL; visual mesh filename=package://arm_description/meshes/axis_0_link.STL
- added link axis_1_link, mass 2.10107115350287; collision mesh filename=package://arm_description/meshes/axis_1_link.STL; visual mesh filename=package://arm_description/meshes/axis_1_link.STL
- added link axis_2_link, mass 3.13644489009951; collision mesh filename=package://arm_description/meshes/axis_2_link.STL; visual mesh filename=package://arm_description/meshes/axis_2_link.STL
- added link ef_carrier_link, mass 0.397605677640027; collision mesh filename=package://arm_description/meshes/ef_carrier_link.STL; visual mesh filename=package://arm_description/meshes/ef_carrier_link.STL
- added link ef_gripper_left_link, mass 0.0813132558225319; collision mesh filename=package://arm_description/meshes/ef_gripper_left_link.STL; visual mesh filename=package://arm_description/meshes/ef_gripper_left_link.STL
- added link ef_gripper_right_link, mass 0.0859306256217421; collision mesh filename=package://arm_description/meshes/ef_gripper_right_link.STL; visual mesh filename=package://arm_description/meshes/ef_gripper_right_link.STL
- added link wrist_box_link, mass 1.95105877103309; collision mesh filename=package://arm_description/meshes/wrist_box_link.STL; visual mesh filename=package://arm_description/meshes/wrist_box_link.STL
- added link wrist_differential_link, mass 0.0655351660884378; collision mesh filename=package://arm_description/meshes/wrist_differential_link.STL; visual mesh filename=package://arm_description/meshes/wrist_differential_link.STL
Joints:
- removed joint Axis_0_Joint
- removed joint Axis_1_Joint
- removed joint Axis_2_Joint
- removed joint Axis_3_Joint
- removed joint Gripper_Slider_Left
- removed joint Gripper_Slider_Right
- removed joint Wrist-EF_Roll_Joint
- removed joint Wrist_Differential_Joint
- added joint axis_0_joint: type revolute, parent base_link, child axis_0_link, origin xyz=0.018772 -0.020734 -0.04971 rpy=1.5708 0 3.1115, axis 0 -1 0, limit lower=-3.14 upper=3.14 effort=0 velocity=31.41593
- added joint axis_1_joint: type revolute, parent axis_0_link, child axis_1_link, origin xyz=-0.0271654135185528 0.0927245490180083 0.00384109909109076 rpy=-3.14159265358977 -0.00524713054608625 1.5707963267949, axis 0 -1 0, limit lower=-1.05 upper=1.6 effort=0 velocity=31.41593
- added joint axis_2_joint: type revolute, parent axis_1_link, child axis_2_link, origin xyz=0.470027000000004 0.0126999999999999 0 rpy=3.14159265358979 0.000449358059257729 0, axis 0 -1 0, limit lower=-2.0 upper=2.0 effort=0 velocity=31.41593
- added joint axis_3_joint: type revolute, parent axis_2_link, child wrist_box_link, origin xyz=0.393826999999998 0 0 rpy=0 -0.000409495780687665 0, axis 0 -1 0, limit lower=-1.6 upper=1.9 effort=0 velocity=31.41593
- added joint ef_gripper_left_joint: type prismatic, parent ef_carrier_link, child ef_gripper_left_link, origin xyz=0 0 -0.031677 rpy=0 0 0, axis 0 -1 0, limit lower=-0.04 upper=0.025 effort=0 velocity=0.015
- added joint ef_gripper_right_joint: type prismatic, parent ef_carrier_link, child ef_gripper_right_link, origin xyz=0 0 -0.031677 rpy=0 0 3.1416, axis 0 1 0, limit lower=-0.025 upper=0.04 effort=0 velocity=0.015, mimic joint=ef_gripper_left_joint multiplier=-1
- added joint wrist_roll_joint: type continuous, parent wrist_differential_link, child ef_carrier_link, origin xyz=0 0.01 0 rpy=-1.5708 -0.21566 -3.1416, axis 0 0 1
- added joint wrist_yaw_joint: type revolute, parent wrist_box_link, child wrist_differential_link, origin xyz=0.176692001200001 -0.00622300000004081 0 rpy=-3.05263944120951 1.57079631189374 1.65994236547327, axis -1 0 0, limit lower=-1.6 upper=1.6 effort=0 velocity=31.41593

File: arm_moveit_config/config/ASTRA_Arm.ros2_control.xacro (robot description, xacro)
@@ -20,57 +20,57 @@
                 </xacro:unless>
             </hardware>
-            <joint name="Axis_0_Joint">
+            <joint name="axis_0_joint">
                 <!-- <command_interface name="position"/> -->
                 <command_interface name="velocity"/>
                 <state_interface name="position">
-                  <param name="initial_value">${initial_positions['Axis_0_Joint']}</param>
+                  <param name="initial_value">${initial_positions['axis_0_joint']}</param>
                 </state_interface>
                 <state_interface name="velocity"/>
             </joint>
-            <joint name="Axis_1_Joint">
+            <joint name="axis_1_joint">
                 <!-- <command_interface name="position"/> -->
                 <command_interface name="velocity"/>
                 <state_interface name="position">
-                  <param name="initial_value">${initial_positions['Axis_1_Joint']}</param>
+                  <param name="initial_value">${initial_positions['axis_1_joint']}</param>
                 </state_interface>
                 <state_interface name="velocity"/>
             </joint>
-            <joint name="Axis_2_Joint">
+            <joint name="axis_2_joint">
                 <!-- <command_interface name="position"/> -->
                 <command_interface name="velocity"/>
                 <state_interface name="position">
-                  <param name="initial_value">${initial_positions['Axis_2_Joint']}</param>
+                  <param name="initial_value">${initial_positions['axis_2_joint']}</param>
                 </state_interface>
                 <state_interface name="velocity"/>
             </joint>
-            <joint name="Axis_3_Joint">
+            <joint name="axis_3_joint">
                 <!-- <command_interface name="position"/> -->
                 <command_interface name="velocity"/>
                 <state_interface name="position">
-                  <param name="initial_value">${initial_positions['Axis_3_Joint']}</param>
+                  <param name="initial_value">${initial_positions['axis_3_joint']}</param>
                 </state_interface>
                 <state_interface name="velocity"/>
             </joint>
-            <joint name="Wrist_Differential_Joint">
+            <joint name="wrist_yaw_joint">
                 <!-- <command_interface name="position"/> -->
                 <command_interface name="velocity"/>
                 <state_interface name="position">
-                  <param name="initial_value">${initial_positions['Wrist_Differential_Joint']}</param>
+                  <param name="initial_value">${initial_positions['wrist_yaw_joint']}</param>
                 </state_interface>
                 <state_interface name="velocity"/>
             </joint>
-            <joint name="Wrist-EF_Roll_Joint">
+            <joint name="wrist_roll_joint">
                 <!-- <command_interface name="position"/> -->
                 <command_interface name="velocity"/>
                 <state_interface name="position">
-                  <param name="initial_value">${initial_positions['Wrist-EF_Roll_Joint']}</param>
+                  <param name="initial_value">${initial_positions['wrist_roll_joint']}</param>
                 </state_interface>
                 <state_interface name="velocity"/>
             </joint>
-            <joint name="Gripper_Slider_Left">
+            <joint name="ef_gripper_left_joint">
                 <command_interface name="position"/>
                 <command_interface name="velocity"/>
                 <state_interface name="position">
-                  <param name="initial_value">${initial_positions['Gripper_Slider_Left']}</param>
+                  <param name="initial_value">${initial_positions['ef_gripper_left_joint']}</param>
                 </state_interface>
                 <state_interface name="velocity"/>

Commit message: refactor!: fix directions on axis 2 & 3

File: arm_description/urdf/ASTRA_Arm.urdf (robot description, URDF)
Before this commit: robot ASTRA_Arm, 9 links, 8 joints
Joints:
- joint axis_2_joint: axis 0 -1 0 -> 0 1 0
- joint axis_3_joint: axis 0 -1 0 -> 0 1 0

Commit message: feat: create rover_description to combine core and arm
Preview in RViz: `ros2 launch rover_description display.launch.py`

Simulate in Gazebo: `ros2 launch rover_description gazebo.launch.py`

File: arm_description/urdf/ASTRA_Arm.urdf (robot description, URDF)
Before this commit: robot ASTRA_Arm, 9 links, 8 joints
Links:
- removed link base_link
- added link arm_base_link, mass 1.344; collision mesh filename=package://arm_description/meshes/base_link.STL; visual mesh filename=package://arm_description/meshes/base_link.STL
Joints:
- joint axis_0_joint: parent base_link -> arm_base_link

File: arm_moveit_config/config/ASTRA_Arm.ros2_control.xacro (robot description, xacro)
@@ -11,5 +11,8 @@
                     <param name="position_state_following_offset">0.0</param>
                 </xacro:if>
-                <xacro:unless value="${hardware_mode == 'mock_components'}">
+                <xacro:if value="${hardware_mode == 'gazebo'}">
+                    <plugin>gz_ros2_control/GazeboSimSystem</plugin>
+                </xacro:if>
+                <xacro:if value="${hardware_mode == 'physical'}">
                     <!-- Use topic_based_ros2_control to interface with anchor and control real hardware -->
                     <plugin>topic_based_ros2_control/TopicBasedSystem</plugin>
@@ -18,5 +21,5 @@
                     <param name="trigger_joint_command_threshold">1e-5</param>  <!-- Set to -1 to disable -->
                     <param name="sum_wrapped_joint_states">false</param>
-                </xacro:unless>
+                </xacro:if>
             </hardware>
             <joint name="axis_0_joint">
@@ -77,4 +80,5 @@
             </joint>
         </ros2_control>
+        <!-- Gazebo ros2_control Plugin tag omitted, arm cannot be ran w/o Core in Gazebo -->
     </xacro:macro>
 </robot>

File: core_description/urdf/core_description.xacro (robot description, xacro)
@@ -2,6 +2,7 @@
 <robot xmlns:xacro="http://www.ros.org/wiki/xacro" name="core_rover">
   <xacro:arg name="hardware_mode" default="gazebo"/>
+  <xacro:arg name="omit_gz_ros2_control" default="false"/>
   <xacro:include filename="core_rover.urdf"/>
   <xacro:include filename="ros2_control.xacro"/>
-  <xacro:core_ros2_control hardware_mode="$(arg hardware_mode)"/>
+  <xacro:core_ros2_control hardware_mode="$(arg hardware_mode)" omit_gz_ros2_control="$(arg omit_gz_ros2_control)"/>
 </robot>

File: core_description/urdf/ros2_control.xacro (robot description, xacro)
@@ -1,5 +1,5 @@
 <?xml version="1.0"?>
 <robot xmlns:xacro="http://www.ros.org/wiki/xacro">
-    <xacro:macro name="core_ros2_control" params="hardware_mode">
+    <xacro:macro name="core_ros2_control" params="hardware_mode omit_gz_ros2_control">
         <ros2_control name="CoreSystem" type="system">
             <hardware>
@@ -40,14 +40,16 @@
             </joint>
         </ros2_control>
-        <xacro:if value="${hardware_mode == 'gazebo'}">
-            <gazebo>
-                <plugin filename="gz_ros2_control-system" name="gz_ros2_control::GazeboSimROS2ControlPlugin">
-                    <parameters>$(find core_description)/config/ros2_controllers.yaml</parameters>
-                    <ros>
-                        <remapping>/diff_controller/cmd_vel_unstamped:=/core/twist</remapping>
-                    </ros>
-                </plugin>
-            </gazebo>
-        </xacro:if>
+        <xacro:unless value="${omit_gz_ros2_control}">
+            <xacro:if value="${hardware_mode == 'gazebo'}">
+                <gazebo>
+                    <plugin filename="gz_ros2_control-system" name="gz_ros2_control::GazeboSimROS2ControlPlugin">
+                        <parameters>$(find core_description)/config/ros2_controllers.yaml</parameters>
+                        <ros>
+                            <remapping>/diff_controller/cmd_vel_unstamped:=/core/twist</remapping>
+                        </ros>
+                    </plugin>
+                </gazebo>
+            </xacro:if>
+        </xacro:unless>
     </xacro:macro>
 </robot>

Commit message: fix(arm): make IK mostly work in Gazebo

File: arm_description/urdf/ASTRA_Arm.urdf (robot description, URDF)
Before this commit: robot ASTRA_Arm, 9 links, 8 joints
Joints:
- joint axis_0_joint: limit lower=-3.14 upper=3.14 effort=0 velocity=31.41593 -> lower=-3.14 upper=3.14 effort=50 velocity=31.41593
- joint axis_1_joint: limit lower=-1.05 upper=1.6 effort=0 velocity=31.41593 -> lower=-1.05 upper=1.6 effort=50 velocity=31.41593
- joint axis_2_joint: limit lower=-2.0 upper=2.0 effort=0 velocity=31.41593 -> lower=-2.0 upper=2.0 effort=50 velocity=31.41593
- joint axis_3_joint: limit lower=-1.6 upper=1.9 effort=0 velocity=31.41593 -> lower=-1.6 upper=1.9 effort=50 velocity=31.41593
- joint ef_gripper_right_joint: limit lower=-0.025 upper=0.04 effort=0 velocity=0.015 -> lower=-0.025 upper=0.04 effort=50 velocity=0.015
- joint wrist_yaw_joint: limit lower=-1.6 upper=1.6 effort=0 velocity=31.41593 -> lower=-1.6 upper=1.6 effort=50 velocity=31.41593

Commit message: feat(arm): add end effector support to IK

File: arm_description/urdf/ASTRA_Arm.urdf (robot description, URDF)
Before this commit: robot ASTRA_Arm, 9 links, 8 joints
Joints:
- joint ef_gripper_left_joint: limit lower=-0.04 upper=0.025 effort=0 velocity=0.015 -> lower=-0.04 upper=0.02 effort=50 velocity=0.015

File: arm_moveit_config/config/ASTRA_Arm.ros2_control.xacro (robot description, xacro)
@@ -72,5 +72,5 @@
             </joint>
             <joint name="ef_gripper_left_joint">
-                <command_interface name="position"/>
+                <!-- <command_interface name="position"/> -->
                 <command_interface name="velocity"/>
                 <state_interface name="position">
